File: parts/alu/arithmetic.kicad_sch (KiCad schematic)
At the start: 38 parts

Commit message: Update High Level
Parts:
- C1, C2, C3, C4, C5: footprint (none) -> Capacitor_SMD:C_0805_2012Metric
- D1, D2, D3, D4, D5, D6, D7, D8: footprint (none) -> LED_THT:LED_D5.0mm
- H1, H2, H3, H4: footprint (none) -> MountingHole:MountingHole_2.2mm_M2_DIN965_Pad
- J1, J2, J5: footprint (none) -> Connector_PinHeader_2.54mm:PinHeader_1x01_P2.54mm_Vertical
- J3, J4, J6, J7: footprint (none) -> Connector_PinHeader_2.54mm:PinHeader_1x08_P2.54mm_Vertical
- J8: footprint (none) -> Connector_PinHeader_2.54mm:PinHeader_1x02_P2.54mm_Vertical
- R1, R2, R3, R4, R5, R6, R7, R8: footprint (none) -> Resistor_SMD:R_0805_2012Metric
- U1, U3: footprint (none) -> Package_DIP:DIP-14_W7.62mm
- U2: footprint (none) -> Package_DIP:DIP-20_W7.62mm
- U4, U5: footprint (none) -> Package_DIP:DIP-16_W7.62mm
