File: parts/clock/clock.kicad_sch (KiCad schematic)
At the start: 32 parts, among them J1 ~CLK, J2 CLK, J3 HLT, J4 PWR, SW1 SW_Push, SW2 SW_SPDT, U1 LM555, U2 LM555, U3 LM555, U4 74HC04, U5 74HC08, U6 74HC32

Commit message: SMD Clock
Parts:
- removed J1: ~CLK, Connector_PinHeader_2.54mm:PinHeader_1x01_P2.54mm_Vertical, symbol Connector_Generic:Conn_01x01
- removed J2: CLK, Connector_PinHeader_2.54mm:PinHeader_1x01_P2.54mm_Vertical, symbol Connector_Generic:Conn_01x01
- removed J3: HLT, Connector_PinHeader_2.54mm:PinHeader_1x01_P2.54mm_Vertical, symbol Connector_Generic:Conn_01x01
- removed J4: PWR, Connector_PinHeader_2.54mm:PinHeader_1x02_P2.54mm_Vertical, symbol Connector_Generic:Conn_01x02
- added J2: Conn_01x08, Connector_IDC:IDC-Header_2x03_P2.54mm_Vertical, symbol Connector_Generic:Conn_01x06
- D1: footprint LED_THT:LED_D5.0mm -> LED_SMD:LED_0805_2012Metric
- U1: renamed from U4; footprint Package_DIP:DIP-14_W7.62mm -> Package_SO:SO-14_3.9x8.65mm_P1.27mm
- U2: renamed from U1; footprint Package_DIP:DIP-8_W7.62mm -> Package_SO:SO-8_3.9x4.9mm_P1.27mm
- U3: renamed from U5; footprint Package_DIP:DIP-14_W7.62mm -> Package_SO:SO-14_3.9x8.65mm_P1.27mm
- U4: renamed from U6; footprint Package_DIP:DIP-14_W7.62mm -> Package_SO:SO-14_3.9x8.65mm_P1.27mm
- U5: renamed from U2; footprint Package_DIP:DIP-8_W7.62mm -> Package_SO:SO-8_3.9x4.9mm_P1.27mm
- U6: renamed from U3; footprint Package_DIP:DIP-8_W7.62mm -> Package_SO:SO-8_3.9x4.9mm_P1.27mm
- renumbered C5 to C1, C6 to C2, C2 to C3, C3 to C4, C4 to C5, C10 to C6, C1 to C7
Connections:
- net CLK: now also J2.2 (Pin_2)
- net GND: now also J2.5 (Pin_5), J2.6 (Pin_6)
- net HLT: now also J2.4 (Pin_4)
- net VCC: now also J2.3 (Pin_3)
- net ~{CLK}: now also J2.1 (Pin_1)
